Commit message: Differential-drive Thorvald (2wd0ws) in gz-sim
- Diff-drive variant is now the default robot (cfg/robot.yaml).
- Propulsion-only drives (type 1) get a fixed steering joint and no
  steering position controller.
- gz-sim: sphere wheel contacts and frictionless ball casters on a
  sprung vertical slide. The springs are soft (2500 N/m, same ~225 N
  preload): at 8000 N/m about 5 cm of terrain twist lifted a drive wheel
  off the ground, so the robot stalled in turns and yawed against the
  command. On the field, achieved yaw rate now tracks the command within
  ~3 % and in-row RMSE on ground truth dropped from 24-31 cm to 2-5 cm.
- twist_to_joints: pure reverse (v < 0, w = 0) commanded steer = pi
  without folding, so the diff-drive robot drove forward. Fold it like
  the turning branch does.
- test_run_control_launch_arguments follows the configured variant.

Co-Authored-By: Claude Opus 5.5 <noreply@anthropic.com>

File: robots/thorvald_model/urdf/thorvald_model.xacro (robot description, xacro)
@@ -199,6 +199,11 @@
       </collision>
     </link>
-    <joint name="${tf_prefix}${steering}" type="revolute">
-      <limit effort="1000" velocity="3" lower="-1.5708" upper="1.5708"/>
+    <!-- type 1 (propulsion only, diff-drive variants) has no steering motor:
+         a revolute joint there just flops under ground forces -->
+    <xacro:property name="drive_type" value="${base_params['motor_drives'][drive].get('type', 0)}" />
+    <joint name="${tf_prefix}${steering}" type="${'fixed' if drive_type == 1 else 'revolute'}">
+      <xacro:unless value="${drive_type == 1}">
+        <limit effort="1000" velocity="3" lower="-1.5708" upper="1.5708"/>
+      </xacro:unless>
       <parent link="${tf_prefix}base_link"/>
 	    <child link="${tf_prefix}${leg}"/>
@@ -221,7 +226,14 @@
 	      <material name="black_material" />
       </visual>
+      <!-- gz-sim: sphere contact. DART's cylinder-vs-triangle-mesh contact on the
+           photogrammetry terrain drops out, so the drive wheels lost traction. -->
       <collision>
         <geometry>
-          <cylinder length="${wheel_width}" radius="${radius_wheel}"/>
+          <xacro:if value="${control_backend == 'gz_sim'}">
+            <sphere radius="${radius_wheel}"/>
+          </xacro:if>
+          <xacro:unless value="${control_backend == 'gz_sim'}">
+            <cylinder length="${wheel_width}" radius="${radius_wheel}"/>
+          </xacro:unless>
         </geometry>
       </collision>
@@ -276,10 +288,32 @@
         </collision>
       </link>
-      <joint name="${tf_prefix}${caster_leg}" type="continuous">
+      <!-- gz-sim: ball casters. The swivelling caster (undamped swivel, placeholder
+           1 kg m^2 wheel inertia) dragged like a brake and made turns asymmetric, so
+           under gz_sim the caster is rigid and its wheel touches the ground through a
+           frictionless sphere. Joints get a _joint suffix: SDF rejects a joint named
+           like a link. -->
+      <!-- The leg slides vertically on a preloaded spring (sits at q=0 under the
+           static load), so on twisted terrain the casters give way instead of
+           lifting a drive wheel off the ground. Keep it soft: the caster load
+           difference is reacted by the drive axle, so at 8000 N/m about 5 cm
+           of terrain twist unloaded a drive wheel on the photogrammetry field.
+           2500 N/m with the rest position 9 cm down keeps the ~225 N preload. -->
+      <xacro:property name="ball_caster" value="${control_backend == 'gz_sim'}" />
+      <joint name="${tf_prefix}${caster_leg}_joint" type="${'prismatic' if ball_caster else 'continuous'}">
         <parent link="${tf_prefix}base_link"/>
       <child link="${tf_prefix}${caster_leg}"/>
       <origin xyz="${x} ${y} ${z}" rpy="0 0 0"/>
         <axis xyz="0 0 1"/>
-      </joint>
+        <xacro:if value="${ball_caster}">
+          <limit lower="-0.1" upper="0.1" effort="10000" velocity="10"/>
+          <dynamics damping="400"/>
+        </xacro:if>
+      </joint>
+      <xacro:if value="${ball_caster}">
+        <gazebo reference="${tf_prefix}${caster_leg}_joint">
+          <springStiffness>2500</springStiffness>
+          <springReference>-0.09</springReference>
+        </gazebo>
+      </xacro:if>
       <link name="${tf_prefix}${caster_wheel}">
         <inertial>
@@ -299,9 +333,20 @@
         <collision>
           <geometry>
-	          <cylinder length="${w_wheel}" radius="${r_wheel}"/>
+            <xacro:if value="${ball_caster}">
+              <sphere radius="${r_wheel}"/>
+            </xacro:if>
+            <xacro:unless value="${ball_caster}">
+	            <cylinder length="${w_wheel}" radius="${r_wheel}"/>
+            </xacro:unless>
           </geometry>
         </collision>
       </link>
-      <joint name="${tf_prefix}${caster_wheel}" type="continuous">
+      <xacro:if value="${ball_caster}">
+        <gazebo reference="${tf_prefix}${caster_wheel}">
+          <mu1>0.0</mu1>
+          <mu2>0.0</mu2>
+        </gazebo>
+      </xacro:if>
+      <joint name="${tf_prefix}${caster_wheel}_joint" type="${'fixed' if ball_caster else 'continuous'}">
         <parent link="${tf_prefix}${caster_leg}"/>
         <child link="${tf_prefix}${caster_wheel}"/>
@@ -779,4 +824,5 @@
     <xacro:if value="${drive in base_params['motor_drives']}">
       <gazebo>
+        <xacro:unless value="${base_params['motor_drives'][drive].get('type', 0) == 1}">
         <plugin filename="gz-sim-joint-position-controller-system"
                 name="gz::sim::systems::JointPositionController">
@@ -791,4 +837,5 @@
           <cmd_min>-60</cmd_min>
         </plugin>
+        </xacro:unless>
       </gazebo>
       <gazebo>
